File: DumbBot.sch (KiCad schematic (older format))
At the start: 10 parts

Commit message: More schema work
Parts:
- added CON?: AVR-ISP-6, AVR-ISP-6, symbol AVR-ISP-6
- added D? (x4): D, symbol D
- added SW?: Switch_SPDT_x2, symbol Switch_SPDT_x2
Other:
- moved on the sheet: U?
Changed lines of the file:
@@
 L DC_Motor U?
 U 1 1 5519B393
-P 7650 1500
-F 0 "U?" H 7650 1300 60  0000 C CNN
-F 1 "DC_Motor" H 7650 1800 60  0000 C CNN
-F 2 "" H 7650 1500 60  0000 C CNN
-F 3 "" H 7650 1500 60  0000 C CNN
-	1    7650 1500
+P 7700 1650
+F 0 "U?" H 7700 1450 60  0000 C CNN
+F 1 "DC_Motor" H 7700 1950 60  0000 C CNN
+F 2 "" H 7700 1650 60  0000 C CNN
+F 3 "" H 7700 1650 60  0000 C CNN
+	1    7700 1650
 	0    -1   -1   0
 $EndComp
@@
 	1    0    0    -1
 $EndComp
+$Comp
+L Switch_SPDT_x2 SW?
+U 1 1 5519B955
+P 8250 2950
+F 0 "SW?" H 8050 3100 50  0000 C CNN
+F 1 "Switch_SPDT_x2" H 8000 2800 50  0000 C CNN
+F 2 "" H 8250 2950 60  0000 C CNN
+F 3 "" H 8250 2950 60  0000 C CNN
+	1    8250 2950
+	1    0    0    -1
+$EndComp
+$Comp
+L AVR-ISP-6 CON?
+U 1 1 5519BA0F
+P 8100 4050
+F 0 "CON?" H 7995 4290 50  0000 C CNN
+F 1 "AVR-ISP-6" H 7835 3820 50  0000 L BNN
+F 2 "AVR-ISP-6" V 7580 4090 50  0001 C CNN
+F 3 "" H 8075 4050 60  0000 C CNN
+	1    8100 4050
+	0    1    1    0
+$EndComp
+$Comp
+L D D?
+U 1 1 5519BC57
+P 7450 2400
+F 0 "D?" H 7450 2500 50  0000 C CNN
+F 1 "D" H 7450 2300 50  0000 C CNN
+F 2 "" H 7450 2400 60  0000 C CNN
+F 3 "" H 7450 2400 60  0000 C CNN
+	1    7450 2400
+	0    1    1    0
+$EndComp
+$Comp
+L D D?
+U 1 1 5519BC5D
+P 7150 2400
+F 0 "D?" H 7150 2500 50  0000 C CNN
+F 1 "D" H 7150 2300 50  0000 C CNN
+F 2 "" H 7150 2400 60  0000 C CNN
+F 3 "" H 7150 2400 60  0000 C CNN
+	1    7150 2400
+	0    -1   -1   0
+$EndComp
+$Comp
+L D D?
+U 1 1 5519BCB5
+P 7150 1300
+F 0 "D?" H 7150 1400 50  0000 C CNN
+F 1 "D" H 7150 1200 50  0000 C CNN
+F 2 "" H 7150 1300 60  0000 C CNN
+F 3 "" H 7150 1300 60  0000 C CNN
+	1    7150 1300
+	0    1    1    0
+$EndComp
+$Comp
+L D D?
+U 1 1 5519BD38
+P 7450 1300
+F 0 "D?" H 7450 1400 50  0000 C CNN
+F 1 "D" H 7450 1200 50  0000 C CNN
+F 2 "" H 7450 1300 60  0000 C CNN
+F 3 "" H 7450 1300 60  0000 C CNN
+	1    7450 1300
+	0    -1   -1   0
+$EndComp
 $EndSCHEMATC
